File: elec/layout/default/spin-dev-board.kicad_pcb (KiCad board)
At the start: 2 copper layers, 225.7 x 100.8 mm, 0 parts

Commit message: layout complete
Parts:
- added C1: Multilayer Ceramic Capacitors MLCC - SMD/SMT 4.7uF 50V 1206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, lib:C1206, F.Cu at (233.1, 94.4)
- added C2: Multilayer Ceramic Capacitors MLCC - SMD/SMT 4.7uF 50V 1206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, lib:C1206, F.Cu at (232.6, 85.8)
- added C3: Multilayer Ceramic Capacitors MLCC - SMD/SMT 220nF 25V 0402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, lib:C0402, F.Cu at (233.3, 89.6)
- added C4: Multilayer Ceramic Capacitors MLCC - SMD/SMT 1uF 6.3V 0402 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, lib:C0402, F.Cu at (228.5, 74.4)
- added C5: Multilayer Ceramic Capacitors MLCC - SMD/SMT 1uF 6.3V 0402 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, lib:C0402, F.Cu at (232.0, 72.8)
- added C6: Multilayer Ceramic Capacitors MLCC - SMD/SMT 100nF 10V 0402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, lib:C0402, F.Cu at (242.7, 101.2)
- added C7: Multilayer Ceramic Capacitors MLCC - SMD/SMT 100nF 10V 0402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, lib:C0402, F.Cu at (239.3, 78.3)
- added DS1: 40V 0.55V@2A 2A SOD-123F Schottky Barrier Diodes (SBD) ROHS, lib:ato-d7ff14dd-2a74-44cb-99b3-1745d3b17ea0, F.Cu at (232.4, 88.0)
- added J1: , lib:CONN-TH_XT30PW-M, F.Cu at (240.8, 110.9)
- added L1: 1A 47uH ±20% SMD Power Inductors ROHS, lib:ato-2d2e488a-5f9f-46bd-846a-d9ea39a9e524, F.Cu at (238.0, 88.8)
- added R1: Chip Resistor - Surface Mount 82KOhms ±5% 1/16W 0402 RoHS, lib:R0402, F.Cu at (230.0, 90.0)
- added R10: Chip Resistor - Surface Mount 0.18Ohms ±5% 1/8W 0805 RoHS, lib:R0805, F.Cu at (243.0, 76.0)
- added R11: Chip Resistor - Surface Mount 20KOhms ±5% 1/16W 0402 RoHS, lib:R0402, F.Cu at (246.6, 105.7)
- added R12: Chip Resistor - Surface Mount 10KOhms ±5% 1/16W 0402 RoHS, lib:R0402, F.Cu at (246.6, 103.7)
- added R13: Chip Resistor - Surface Mount 20KOhms ±5% 1/16W 0402 RoHS, lib:R0402, F.Cu at (246.8, 71.0)
- added R14: Chip Resistor - Surface Mount 10KOhms ±5% 1/16W 0402 RoHS, lib:R0402, F.Cu at (246.8, 73.1)
- added R2: Chip Resistor - Surface Mount 11KOhms ±5% 1/16W 0402 RoHS, lib:R0402, F.Cu at (230.0, 92.0)
- added R3: Chip Resistor - Surface Mount 1KOhms ±5% 1/16W 0402 RoHS, lib:R0402, F.Cu at (250.8, 85.1)
- added R4: Chip Resistor - Surface Mount 1KOhms ±5% 1/16W 0402 RoHS, lib:R0402, F.Cu at (250.8, 87.6)
- added R5: Chip Resistor - Surface Mount 1KOhms ±5% 1/16W 0402 RoHS, lib:R0402, F.Cu at (250.8, 90.2)
- added R6: Chip Resistor - Surface Mount 1KOhms ±5% 1/16W 0402 RoHS, lib:R0402, F.Cu at (250.8, 92.7)
- added R7: Chip Resistor - Surface Mount 18KOhms ±5% 1/16W 0402 RoHS, lib:R0402, F.Cu at (233.6, 74.0)
- added R8: Chip Resistor - Surface Mount 10KOhms ±5% 1/16W 0402 RoHS, lib:R0402, F.Cu at (233.6, 76.0)
- added R9: Chip Resistor - Surface Mount 0.18Ohms ±5% 1/8W 0805 RoHS, lib:R0805, F.Cu at (237.0, 102.4)
- added U1: , lib:SOT-23-6_L2.9-W1.6-P0.95-LS2.8-BR, F.Cu at (232.9, 91.7)
- added U2: , lib:HDR-SMD_8P-P2.54-V-M-R2-C4-LS7.4, F.Cu at (256.5, 88.9)
- added U3: , lib:SOT-23-5_L3.0-W1.7-P0.95-LS2.8-BL, F.Cu at (231.1, 74.9)
- added U4: , lib:CONN-TH_XT30PW-F-1, F.Cu at (240.7, 69.0)
- added U5: , lib:SOT-23-6_L2.9-W1.6-P0.95-LS2.8-TL, F.Cu at (240.2, 101.8)
- added U6: , lib:SOT-23-6_L2.9-W1.6-P0.95-LS2.8-TL, F.Cu at (240.0, 76.2)
Routing:
- net gnd: track 0.00 -> 121.5 mm, vias 0 -> 7
- net vcc-3: track 0.00 -> 44.4 mm, vias 0 -> 3
- net vcc-1: track 0.00 -> 41.7 mm
- net vcc: track 0.00 -> 27.8 mm
- net io-2: track 0.00 -> 19.9 mm
- net io-3: track 0.00 -> 17.1 mm, vias 0 -> 2
- net io-1: track 0.00 -> 16.5 mm
- net io-4: track 0.00 -> 14.0 mm
- net SW: track 0.00 -> 6.90 mm
- net gnd-2: track 0.00 -> 5.57 mm
- net gnd-1: track 0.00 -> 5.42 mm
- net io: track 0.00 -> 2.91 mm
- net io-5: track 0.00 -> 2.46 mm
- net vcc-2: track 0.00 -> 1.73 mm
Other:
- outline, holes or cut-outs redrawn
